Commit message: func

File: machine_tool/machine_tool_description/urdf/xacro/main.xacro (robot description, xacro)
@@ -160,5 +160,5 @@
       <visual>
         <geometry>
-          <mesh filename="package://machine_tool_description/meshes/iphone/iPhone.stl" scale = "0.001 0.001 0.001" />
+          <mesh filename="package://machine_tool_description/meshes/iphone/test_model.STL" scale = "0.001 0.001 0.001" />
         </geometry>
         <material name="LightGrey">
@@ -180,5 +180,5 @@
     </link>
     <joint name="plate_joine" type="fixed">
-        <origin xyz="0 0 0.03" rpy="0 0 0"></origin>
+        <origin xyz="0 0 0" rpy="0 0 0"></origin>
         <parent link="plate" />
         <child link="iphone"/>

Commit message: check

File: machine_tool/machine_tool_description/urdf/xacro/main.xacro (robot description, xacro)
@@ -180,5 +180,5 @@
     </link>
     <joint name="plate_joine" type="fixed">
-        <origin xyz="0 0 0" rpy="0 0 0"></origin>
+        <origin xyz="-0.0358 0.07353 0" rpy="1.5707963 0 0"></origin>
         <parent link="plate" />
         <child link="iphone"/>
