Commit message: new

File: machine_tool/machine_tool_description/urdf/xacro/main_pose.xacro (robot description, xacro)
@@ -155,5 +155,5 @@
         <child link="plate"/>
         <axis xyz="0 0 1" />
-        <limit effort="30" velocity="100.0" lower="-6.28" upper="6.28" />
+        <limit effort="30" velocity="100.0" lower="-20" upper="20" />
     </joint>
     <link name="iphone">
@@ -255,8 +255,8 @@
       <type>transmission_interface/SimpleTransmission</type>
       <joint name="x_joint">
-      <hardwareInterface>hardware_interface/VelocityJointInterface</hardwareInterface>
+      <hardwareInterface>hardware_interface/PositionJointInterface</hardwareInterface>
       </joint>
       <actuator name="x_joint_motor">
-      <hardwareInterface>hardware_interface/VelocityJointInterface</hardwareInterface>
+      <hardwareInterface>hardware_interface/PositionJointInterface</hardwareInterface>
         <mechanicalReduction>1</mechanicalReduction>
       </actuator>
@@ -265,8 +265,8 @@
       <type>transmission_interface/SimpleTransmission</type>
       <joint name="y_joint">
-      <hardwareInterface>hardware_interface/VelocityJointInterface</hardwareInterface>
+      <hardwareInterface>hardware_interface/PositionJointInterface</hardwareInterface>
       </joint>
       <actuator name="y_joint_motor">
-      <hardwareInterface>hardware_interface/VelocityJointInterface</hardwareInterface>
+      <hardwareInterface>hardware_interface/PositionJointInterface</hardwareInterface>
         <mechanicalReduction>1</mechanicalReduction>
       </actuator>
@@ -275,8 +275,8 @@
       <type>transmission_interface/SimpleTransmission</type>
       <joint name="r_joint">
-      <hardwareInterface>hardware_interface/VelocityJointInterface</hardwareInterface>
+      <hardwareInterface>hardware_interface/PositionJointInterface</hardwareInterface>
       </joint>
       <actuator name="r_joint_motor">
-      <hardwareInterface>hardware_interface/VelocityJointInterface</hardwareInterface>
+      <hardwareInterface>hardware_interface/PositionJointInterface</hardwareInterface>
         <mechanicalReduction>1</mechanicalReduction>
       </actuator>
